Commit message: Working ish with arm

File: crx_description/urdf/crx10ia_l/crx10ia_l.urdf.xacro (robot description, xacro)
@@ -44,16 +44,16 @@
     <xacro:property name="j5_v" value="180"/>
     <xacro:property name="j6_v" value="180"/>
-    <xacro:property name="j1_u" value="179.9"/>
-    <xacro:property name="j2_u" value="179.9"/>
-    <xacro:property name="j3_u" value="270"/>
-    <xacro:property name="j4_u" value="190"/>
-    <xacro:property name="j5_u" value="179.9"/>
-    <xacro:property name="j6_u" value="225"/>
-    <xacro:property name="j1_l" value="-179.9"/>
-    <xacro:property name="j2_l" value="-179.9"/>
-    <xacro:property name="j3_l" value="-270"/>
-    <xacro:property name="j4_l" value="-190"/>
-    <xacro:property name="j5_l" value="-179.9"/>
-    <xacro:property name="j6_l" value="-225"/>
+    <xacro:property name="j1_u" value="175"/>
+    <xacro:property name="j2_u" value="175"/>
+    <xacro:property name="j3_u" value="265"/>
+    <xacro:property name="j4_u" value="175"/>
+    <xacro:property name="j5_u" value="175"/>
+    <xacro:property name="j6_u" value="220"/>
+    <xacro:property name="j1_l" value="-175"/>
+    <xacro:property name="j2_l" value="-175"/>
+    <xacro:property name="j3_l" value="-265"/>
+    <xacro:property name="j4_l" value="-175"/>
+    <xacro:property name="j5_l" value="-175"/>
+    <xacro:property name="j6_l" value="-220"/>
     <xacro:property name="mz_1" value="0.1277"/>
     <xacro:property name="mz_2" value="0.245"/>

Commit message: Reachability tests

File: crx_description/urdf/crx10ia_l/crx10ia_l.urdf.xacro (robot description, xacro)
@@ -52,5 +52,5 @@
     <xacro:property name="j1_l" value="-175"/>
     <xacro:property name="j2_l" value="-175"/>
-    <xacro:property name="j3_l" value="-265"/>
+    <xacro:property name="j3_l" value="-85"/>
     <xacro:property name="j4_l" value="-175"/>
     <xacro:property name="j5_l" value="-175"/>
